Commit message: [urdf] Use obj as collision meshes for the hands, and tweaked tool frames.

File: urdf/armar6.urdf (robot description, URDF)
Before this commit: robot Armar6, 59 links, 58 joints
Links:
- link Hand L Palm: geometry collision mesh filename=package://armar6_description/mesh/obj/collision/hand_v3/pal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 scale=1.00000 1.00000 1.00000; visual mesh filename=package://armar6_description/mesh/stl/visual/hand_v3/palm_l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 scale=1.00000 1.00000 1.00000
- link Hand R Palm: geometry collision mesh filename=package://armar6_description/mesh/obj/collision/hand_v3/pal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 scale=1.00000 1.00000 1.00000; visual mesh filename=package://armar6_description/mesh/stl/visual/hand_v3/palm_r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 scale=1.00000 1.00000 1.00000
- link Index L 1: geometry collision mesh filename=package://armar6_description/mesh/obj/collision/hand_v3/ind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 scale=1.00000 1.00000 1.00000; visual mesh filename=package://armar6_description/mesh/stl/visual/hand_v3/index_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 scale=1.00000 1.00000 1.00000
- link Index L 2: geometry collision mesh filename=package://armar6_description/mesh/obj/collision/hand_v3/ind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 scale=1.00000 1.00000 1.00000; visual mesh filename=package://armar6_description/mesh/stl/visual/hand_v3/index_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 scale=1.00000 1.00000 1.00000
- link Index L 3: geometry collision mesh filename=package://armar6_description/mesh/obj/collision/hand_v3/ind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 scale=1.00000 1.00000 1.00000; visual mesh filename=package://armar6_description/mesh/stl/visual/hand_v3/index_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 scale=1.00000 1.00000 1.00000
- link Index R 1: geometry collision mesh filename=package://armar6_description/mesh/obj/collision/hand_v3/ind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 scale=1.00000 1.00000 1.00000; visual mesh filename=package://armar6_description/mesh/stl/visual/hand_v3/index_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 scale=1.00000 1.00000 1.00000
- link Index R 2: geometry collision mesh filename=package://armar6_description/mesh/obj/collision/hand_v3/ind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 scale=1.00000 1.00000 1.00000; visual mesh filename=package://armar6_description/mesh/stl/visual/hand_v3/index_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 scale=1.00000 1.00000 1.00000
- link Index R 3: geometry collision mesh filename=package://armar6_description/mesh/obj/collision/hand_v3/ind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 scale=1.00000 1.00000 1.00000; visual mesh filename=package://armar6_description/mesh/stl/visual/hand_v3/index_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 scale=1.00000 1.00000 1.00000
- link Middle L 1: geometry collision mesh filename=package://armar6_description/mesh/obj/collision/hand_v3/mid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 scale=1.00000 1.00000 1.00000; visual mesh filename=package://armar6_description/mesh/stl/visual/hand_v3/middle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 scale=1.00000 1.00000 1.00000
- link Middle L 2: geometry collision mesh filename=package://armar6_description/mesh/obj/collision/hand_v3/mid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 scale=1.00000 1.00000 1.00000; visual mesh filename=package://armar6_description/mesh/stl/visual/hand_v3/middle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 scale=1.00000 1.00000 1.00000
- link Middle L 3: geometry collision mesh filename=package://armar6_description/mesh/obj/collision/hand_v3/mid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 scale=1.00000 1.00000 1.00000; visual mesh filename=package://armar6_description/mesh/stl/visual/hand_v3/middle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 scale=1.00000 1.00000 1.00000
- link Middle R 1: geometry collision mesh filename=package://armar6_description/mesh/obj/collision/hand_v3/mid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 scale=1.00000 1.00000 1.00000; visual mesh filename=package://armar6_description/mesh/stl/visual/hand_v3/middle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 scale=1.00000 1.00000 1.00000
- link Middle R 2: geometry collision mesh filename=package://armar6_description/mesh/obj/collision/hand_v3/mid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 scale=1.00000 1.00000 1.00000; visual mesh filename=package://armar6_description/mesh/stl/visual/hand_v3/middle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 scale=1.00000 1.00000 1.00000
- link Middle R 3: geometry collision mesh filename=package://armar6_description/mesh/obj/collision/hand_v3/mid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 scale=1.00000 1.00000 1.00000; visual mesh filename=package://armar6_description/mesh/stl/visual/hand_v3/middle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 scale=1.00000 1.00000 1.00000
- link Pinky L 1: geometry collision mesh filename=package://armar6_description/mesh/obj/collision/hand_v3/pin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 scale=1.00000 1.00000 1.00000; visual mesh filename=package://armar6_description/mesh/stl/visual/hand_v3/pinky_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 scale=1.00000 1.00000 1.00000
- link Pinky L 2: geometry collision mesh filename=package://armar6_description/mesh/obj/collision/hand_v3/pin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 scale=1.00000 1.00000 1.00000; visual mesh filename=package://armar6_description/mesh/stl/visual/hand_v3/pinky_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 scale=1.00000 1.00000 1.00000
- link Pinky L 3: geometry collision mesh filename=package://armar6_description/mesh/obj/collision/hand_v3/pin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 scale=1.00000 1.00000 1.00000; visual mesh filename=package://armar6_description/mesh/stl/visual/hand_v3/pinky_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 scale=1.00000 1.00000 1.00000
- link Pinky R 1: geometry collision mesh filename=package://armar6_description/mesh/obj/collision/hand_v3/pin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 scale=1.00000 1.00000 1.00000; visual mesh filename=package://armar6_description/mesh/stl/visual/hand_v3/pinky_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 scale=1.00000 1.00000 1.00000
- link Pinky R 2: geometry collision mesh filename=package://armar6_description/mesh/obj/collision/hand_v3/pin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 scale=1.00000 1.00000 1.00000; visual mesh filename=package://armar6_description/mesh/stl/visual/hand_v3/pinky_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 scale=1.00000 1.00000 1.00000
- link Pinky R 3: geometry collision mesh filename=package://armar6_description/mesh/obj/collision/hand_v3/pin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 scale=1.00000 1.00000 1.00000; visual mesh filename=package://armar6_description/mesh/stl/visual/hand_v3/pinky_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 scale=1.00000 1.00000 1.00000
- link Ring L 1: geometry collision mesh filename=package://armar6_description/mesh/obj/collision/hand_v3/rin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 scale=1.00000 1.00000 1.00000; visual mesh filename=package://armar6_description/mesh/stl/visual/hand_v3/ring_p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 scale=1.00000 1.00000 1.00000
- link Ring L 2: geometry collision mesh filename=package://armar6_description/mesh/obj/collision/hand_v3/rin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 scale=1.00000 1.00000 1.00000; visual mesh filename=package://armar6_description/mesh/stl/visual/hand_v3/ring_i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 scale=1.00000 1.00000 1.00000
- link Ring L 3: geometry collision mesh filename=package://armar6_description/mesh/obj/collision/hand_v3/rin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 scale=1.00000 1.00000 1.00000; visual mesh filename=package://armar6_description/mesh/stl/visual/hand_v3/ring_d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 scale=1.00000 1.00000 1.00000
- link Ring R 1: geometry collision mesh filename=package://armar6_description/mesh/obj/collision/hand_v3/rin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 scale=1.00000 1.00000 1.00000; visual mesh filename=package://armar6_description/mesh/stl/visual/hand_v3/ring_p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 scale=1.00000 1.00000 1.00000
- link Ring R 2: geometry collision mesh filename=package://armar6_description/mesh/obj/collision/hand_v3/rin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 scale=1.00000 1.00000 1.00000; visual mesh filename=package://armar6_description/mesh/stl/visual/hand_v3/ring_i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 scale=1.00000 1.00000 1.00000
- link Ring R 3: geometry collision mesh filename=package://armar6_description/mesh/obj/collision/hand_v3/rin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 scale=1.00000 1.00000 1.00000; visual mesh filename=package://armar6_description/mesh/stl/visual/hand_v3/ring_d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 scale=1.00000 1.00000 1.00000
- link Thumb L 1: geometry collision mesh filename=package://armar6_description/mesh/obj/collision/hand_v3/thu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 scale=1.00000 1.00000 1.00000; visual mesh filename=package://armar6_description/mesh/stl/visual/hand_v3/thumb_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 scale=1.00000 1.00000 1.00000
- link Thumb L 2: geometry collision mesh filename=package://armar6_description/mesh/obj/collision/hand_v3/thu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 scale=1.00000 1.00000 1.00000; visual mesh filename=package://armar6_description/mesh/stl/visual/hand_v3/thumb_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 scale=1.00000 1.00000 1.00000
- link Thumb R 1: geometry collision mesh filename=package://armar6_description/mesh/obj/collision/hand_v3/thu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 scale=1.00000 1.00000 1.00000; visual mesh filename=package://armar6_description/mesh/stl/visual/hand_v3/thumb_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 scale=1.00000 1.00000 1.00000
- link Thumb R 2: geometry collision mesh filename=package://armar6_description/mesh/obj/collision/hand_v3/thu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 scale=1.00000 1.00000 1.00000; visual mesh filename=package://armar6_description/mesh/stl/visual/hand_v3/thumb_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 scale=1.00000 1.00000 1.00000
Joints:
- joint left_tool_frame_joint: origin xyz=0.15 -0.1 0.01 rpy=1.57 0 0 -> xyz=0.15 -0.08 0.01 rpy=1.57 0 0.7854
- joint right_tool_frame_joint: origin xyz=0.15 -0.1 -0.01 rpy=1.57 0 0 -> xyz=0.15 -0.08 -0.01 rpy=1.57 0 0.7854

Commit message: [urdf] tweak for tool frames

File: urdf/armar6.urdf (robot description, URDF)
Before this commit: robot Armar6, 59 links, 58 joints
Joints:
- joint left_tool_frame_joint: origin xyz=0.15 -0.08 0.01 rpy=1.57 0 0.7854 -> xyz=0.15 -0.07 0.01 rpy=1.57 0 0.7854
- joint right_tool_frame_joint: origin xyz=0.15 -0.08 -0.01 rpy=1.57 0 0.7854 -> xyz=0.15 -0.07 -0.01 rpy=1.57 0 0.7854
